File: Line_kicad/line_f/line_f.kicad_sch (KiCad schematic)
At the start: 16 parts, among them M2 Motor_DC, M3 Motor_DC, SW1 SW_SPST, SW2 SW_SPDT, SW3 SW_Push, SW4 SW_Push, U1 TB6612FNG_LINE, m1 BLACKPILL

Commit message: 3#
Parts:
- BT1: footprint Connector_AMASS:AMASS_XT60-M_1x02_P7.20mm_Vertical -> LINE_F_FOOT_LIB:BATTERY_LINE_XT60
Changed lines of the file:
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@@
 			)
 		)
-		(property "Footprint" "Connector_AMASS:AMASS_XT60-M_1x02_P7.20mm_Vertical"
+		(property "Footprint" "LINE_F_FOOT_LIB:BATTERY_LINE_XT60"
 			(at 81.026 121.92 90)
 			(effects

Commit message: 3#
Connections:
- net BI2: now also m1.17 (B9); no longer m1.13 (B5)
- net JPULSE: now also m1.34 (A1); no longer m1.5 (A8)
- net PWMA: now also m1.33 (A2); no longer m1.35 (A0)
- net PWMB: now also m1.5 (A8); no longer m1.34 (A1)
- no-connect marks 10 -> 13

Commit message: 3#
Other:
- note added: "Verified"
Changed lines of the file:
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@@
+		)
+	)
+	(text "Verified\n"
+		(exclude_from_sim no)
+		(at 39.37 67.31 0)
+		(effects
+			(font
+				(size 1.27 1.27)
+			)
 		)
 	)

Commit message: 3#
Parts:
- U1: footprint LINE_F_FOOT_LIB:TB6612FNG_LINE -> ROB-14450:MODULE_ROB-14450
Connections:
- no-connect marks 13 -> 5
Changed lines of the file:
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@@
 	)
 	(no_connect
-		(at 190.5 143.51)
-	)
-	(no_connect
 		(at 246.38 100.33)
 	)
@@
 	)
 	(no_connect
-		(at 190.5 133.35)
-	)
-	(no_connect
-		(at 190.5 146.05)
-	)
-	(no_connect
-		(at 190.5 138.43)
-	)
-	(no_connect
-		(at 190.5 140.97)
-	)
-	(no_connect
-		(at 190.5 107.95)
-	)
-	(no_connect
-		(at 162.56 128.27)
-	)
-	(no_connect
-		(at 190.5 135.89)
-	)
-	(no_connect
 		(at 246.38 97.79)
 	)
@@
 		)
 	)
+	(text "Verified\n"
+		(exclude_from_sim no)
+		(at 126.238 74.676 0)
+		(effects
+			(font
+				(size 1.27 1.27)
+			)
+		)
+	)
+	(text "Verified\n"
+		(exclude_from_sim no)
+		(at 81.28 83.312 0)
+		(effects
+			(font
+				(size 1.27 1.27)
+			)
+		)
+	)
+	(text "Verified\n"
+		(exclude_from_sim no)
+		(at 172.974 60.96 0)
+		(effects
+			(font
+				(size 1.27 1.27)
+			)
+		)
+	)
 	(text "SWITCHES\n"
 		(exclude_from_sim no)
@@
 		)
 	)
+	(text "Verified\n"
+		(exclude_from_sim no)
+		(at 232.41 68.58 0)
+		(effects
+			(font
+				(size 1.27 1.27)
+			)
+		)
+	)
 	(global_label "SW_TRY"
 		(shape input)
@@
 			)
 		)
-		(property "Footprint" "LINE_F_FOOT_LIB:TB6612FNG_LINE"
+		(property "Footprint" "ROB-14450:MODULE_ROB-14450"
 			(at 231.14 92.71 0)
 			(effects

Commit message: 3#
Parts:
- U1: footprint ROB-14450:MODULE_ROB-14450 -> LINE_F_FOOT_LIB:TB6612FNG_LINE
Changed lines of the file:
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@@
 			)
 		)
-		(property "Footprint" "ROB-14450:MODULE_ROB-14450"
+		(property "Footprint" "LINE_F_FOOT_LIB:TB6612FNG_LINE"
 			(at 231.14 92.71 0)
 			(effects
