File: Line_kicad/line_f/line_f.kicad_pcb (KiCad board)
At the start: 2 copper layers, 135 x 157.5 mm, 16 parts, among them M2 Motor_DC, M3 Motor_DC, SW1 SW_SPST, SW2 SW_SPDT, SW3 SW_Push, SW4 SW_Push, U1 TB6612FNG_LINE, m1 BLACKPILL

Commit message: 3#
Parts:
- moved LSA_UART1 99.0 mm to (144.2, 185.6)
- moved SW1 89.1 mm to (41.5, 176.8)
- moved SW3 87.8 mm to (36.0, 126.9)
- moved D1 79.6 mm to (72.0, 132.0)
- moved SW2 74.9 mm to (66.0, 127.5), turned to 90 degrees
- moved m1 72.7 mm to (119.9, 145.5), turned to 180 degrees
- moved LSA_ANALOG1 71.2 mm to (96.7, 178.2)
- moved SW4 66.9 mm to (51.0, 126.9)
- moved BUCK1 52.4 mm to (45.8, 171.4), turned to 180 degrees
- moved R1 43.2 mm to (91.7, 124.7), turned to 0 degrees
- moved LSA_DIGITAL1 35.6 mm to (122.0, 182.7)
- moved BT1 24.2 mm to (85.4, 136.0)
- moved U1 18.3 mm to (60.9, 147.8)
- moved M2 16.7 mm to (37.4, 150.6)
- moved MPU1 14.4 mm to (95.8, 145.7), turned to 180 degrees
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Connections:
- M2 pad 1: AO1 -> (no net)
- M2 pad 2: AO2 -> (no net)
- M3 pad 1: BO1 -> (no net)
- M3 pad 2: BO2 -> (no net)
Other:
- board size 135 x 157.5 mm -> 136.5 x 161.5 mm

Commit message: 3#
Parts:
- moved SW4 102.8 mm to (141.0, 176.6)
- moved SW3 100.4 mm to (123.5, 176.1)
- moved LSA_ANALOG1 85.5 mm to (161.8, 122.7)
- moved m1 78.5 mm to (90.9, 72.5), turned to 0 degrees
- moved LSA_DIGITAL1 74.3 mm to (72.6, 127.1)
- moved U1 66.0 mm to (126.5, 155.0)
- moved R1 62.6 mm to (57.8, 177.3)
- moved SW2 59.8 mm to (31.9, 176.6), turned to 0 degrees
- moved LSA_UART1 56.5 mm to (136.2, 129.6)
- moved D1 56.1 mm to (31.9, 171.3)
- moved SW1 44.9 mm to (35.5, 132.3)
- moved BT1 30.5 mm to (87.3, 105.6)
- moved BUCK1 21.6 mm to (48.3, 149.9)
- moved MPU1 7.52 mm to (98.1, 138.5)
- moved M2 3.40 mm to (34.0, 150.4)
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Other:
- board size 136.5 x 161.5 mm -> 179.7 x 172.5 mm

Commit message: Update line_f.kicad_pcb
Parts:
- moved MPU1 27.0 mm to (83.2, 161.1), turned to 0 degrees
- moved BUCK1 16.9 mm to (64.2, 156.0), turned to 0 degrees
- moved U1 4.69 mm to (126.4, 150.3)
- moved SW2 3.90 mm to (34.5, 179.5)
- moved M3 1.44 mm to (142.5, 152.4)
- moved SW3 0.62 mm to (124.0, 176.5)

Commit message: 3#
Parts:
- added M2: Motor_DC, LINE_F_FOOT_LIB:connector_motor, F.Cu at (4.38, 7.43)
- added M3: Motor_DC, LINE_F_FOOT_LIB:connector_motor, F.Cu at (4.38, 16.1)
Connections:
- SW2 pad 3: 5V -> S_3V3
- m1 pad 16: unconnected-(m1-B8-Pad16) -> D6
- m1 pad 25: D6 -> unconnected-(m1-B2-Pad25)

Commit message: 3#
Parts:
- removed the M2 at (34.0, 150.4)
- removed the M3 at (142.5, 152.4)
- moved M2 205.0 mm to (149.5, 152.2), turned to 90 degrees
- moved M3 138.5 mm to (34.5, 151.3), turned to -90 degrees

Commit message: 3#
Routing:
- net C_GND: track 0.00 -> 358.5 mm, vias 0 -> 1
- net S_3V3: track 0.00 -> 212.5 mm, vias 0 -> 1
- net SW_TRY: track 0.00 -> 176.7 mm, vias 0 -> 1
- net SW_RUN: track 0.00 -> 161.0 mm, vias 0 -> 1
- net V_BAT: track 0.00 -> 159.5 mm, vias 0 -> 1
- net 5V: track 0.00 -> 154.6 mm, vias 0 -> 2
- net PRIORITY_SW: track 0.00 -> 153.8 mm, vias 0 -> 1
- net STBY: track 0.00 -> 140.8 mm, vias 0 -> 2
- net LED_F: track 0.00 -> 135.2 mm
- net BI2: track 0.00 -> 126.0 mm, vias 0 -> 2
- net JPULSE: track 0.00 -> 125.1 mm, vias 0 -> 1
- net AI2: track 0.00 -> 122.5 mm, vias 0 -> 1
- net AI1: track 0.00 -> 119.8 mm, vias 0 -> 1
- net BI1: track 0.00 -> 118.4 mm, vias 0 -> 1
- net D7: track 0.00 -> 114.2 mm, vias 0 -> 1
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
Commit message: 3#
Routing:
- net C_GND: track 358.5 -> 0.00 mm, vias 1 -> 0
- net S_3V3: track 212.5 -> 0.00 mm, vias 1 -> 0
- net SW_TRY: track 176.7 -> 0.00 mm, vias 1 -> 0
- net SW_RUN: track 161.0 -> 0.00 mm, vias 1 -> 0
- net V_BAT: track 159.5 -> 0.00 mm, vias 1 -> 0
- net 5V: track 154.6 -> 0.00 mm, vias 2 -> 0
- net PRIORITY_SW: track 153.8 -> 0.00 mm, vias 1 -> 0
- net STBY: track 140.8 -> 0.00 mm, vias 2 -> 0
- net LED_F: track 135.2 -> 0.00 mm
- net BI2: track 126.0 -> 0.00 mm, vias 2 -> 0
- net JPULSE: track 125.1 -> 0.00 mm, vias 1 -> 0
- net AI2: track 122.5 -> 0.00 mm, vias 1 -> 0
- net AI1: track 119.8 -> 0.00 mm, vias 1 -> 0
- net BI1: track 118.4 -> 0.00 mm, vias 1 -> 0
- net D7: track 114.2 -> 0.00 mm, vias 1 -> 0
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