File: Line_kicad/line_f/line_f.kicad_pcb (KiCad board)
At the start: 2 copper layers, 137.5 x 170 mm, 16 parts, among them M2 Motor_DC, M3 Motor_DC, SW1 SW_SPST, SW2 SW_SPDT, SW3 SW_Push, SW4 SW_Push, U1 TB6612FNG_LINE, m1 BLACKPILL

Commit message: 3#
Other:
- board text added: "BTZ"
- board text added: "Run"
Changed lines of the file:
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@@
 			(at 3.6 -5.3 0)
 			(layer "F.SilkS")
+			(hide yes)
 			(effects
 				(font
@@
 			(unlocked yes)
 			(layer "F.SilkS")
+			(hide yes)
 			(effects
 				(font
@@
 			(at -0.04 -23.9 0)
 			(layer "F.SilkS")
+			(hide yes)
 			(effects
 				(font
@@
 			(unlocked yes)
 			(layer "F.SilkS")
+			(hide yes)
 			(effects
 				(font
@@
 			(at 0.06 5.17 90)
 			(layer "F.SilkS")
+			(hide yes)
 			(effects
 				(font
@@
 			(unlocked yes)
 			(layer "F.SilkS")
+			(hide yes)
 			(effects
 				(font
@@
 		(layer "Edge.Cuts")
 	)
+	(gr_text "Run"
+		(at 154 183.5 0)
+		(layer "F.Cu")
+		(effects
+			(font
+				(size 1.5 1.5)
+				(thickness 0.3)
+				(bold yes)
+			)
+			(justify left bottom)
+		)
+	)
+	(gr_text "BTZ"
+		(at 140 184 0)
+		(layer "F.SilkS")
+		(effects
+			(font
+				(size 1 1)
+				(thickness 0.1)
+			)
+			(justify left bottom)
+		)
+	)
 	(group ""

Commit message: 3#
Other:
- board text added: "Run2'"
Changed lines of the file:
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@@
+		)
+	)
+	(gr_text "Run2'"
+		(at 154.5 180 0)
+		(layer "F.Mask")
+		(effects
+			(font
+				(size 1 1)
+				(thickness 0.15)
+			)
+			(justify left bottom)
 		)
 	)

Commit message: 3#
Parts:
- BT1: footprint Connector_AMASS:AMASS_XT60-M_1x02_P7.20mm_Vertical -> LINE_F_FOOT_LIB:BATTERY_LINE_XT60
- moved BT1 9.00 mm to (93.0, 112.5)
Changed lines of the file:
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@@
 	(net 62 "unconnected-(U1-GND-Pad8)")
 	(net 63 "unconnected-(U1-GND-Pad3)")
-	(footprint "Connector_AMASS:AMASS_XT60-M_1x02_P7.20mm_Vertical"
+	(footprint "LINE_F_FOOT_LIB:BATTERY_LINE_XT60"
 		(layer "F.Cu")
-		(at 87.3 105.58)
-		(descr "AMASS female XT60, through hole, vertical, https://www.tme.eu/Document/2d152ced3b7a446066e6c419d84bb460/XT60%20SPEC.pdf")
-		(tags "XT60 female vertical")
+		(at 93 112.55)
 		(property "Reference" "BT1"
-			(at 3.6 -5.3 0)
-			(layer "F.SilkS")
-			(hide yes)
-			(effects
-				(font
-					(size 1 1)
-					(thickness 0.15)
+			(at 0 -0.5 0)
+			(unlocked yes)
+			(layer "F.SilkS")
+			(hide yes)
+			(effects
+				(font
+					(size 1 1)
+					(thickness 0.1)
 				)
 			)
 		)
 		(property "Value" "Battery"
-			(at 3.6 5.4 0)
-			(layer "F.Fab")
-			(effects
-				(font
-					(size 1 1)
-					(thickness 0.15)
-				)
-			)
-		)
-		(property "Footprint" "Connector_AMASS:AMASS_XT60-M_1x02_P7.20mm_Vertical"
+			(at 0 1 0)
+			(unlocked yes)
+			(layer "F.Fab")
+			(effects
+				(font
+					(size 1 1)
+					(thickness 0.15)
+				)
+			)
+		)
+		(property "Footprint" "LINE_F_FOOT_LIB:BATTERY_LINE_XT60"
 			(at 0 0 0)
 			(unlocked yes)
@@
 			(effects
 				(font
-					(size 1.27 1.27)
+					(size 1 1)
 					(thickness 0.15)
 				)
@@
 			(effects
 				(font
-					(size 1.27 1.27)
+					(size 1 1)
 					(thickness 0.15)
 				)
@@
 			(effects
 				(font
-					(size 1.27 1.27)
+					(size 1 1)
 					(thickness 0.15)
 				)
@@
 		(attr through_hole)
 		(fp_line
-			(start -4.25 -1.6)
-			(end -4.25 1.55)
-			(stroke
-				(width 0.12)
-				(type solid)
-			)
-			(layer "F.SilkS")
-		)
-		(fp_line
-			(start -4.25 1.55)
-			(end -1.4 4.15)
-			(stroke
-				(width 0.12)
-				(type solid)
-			)
-			(layer "F.SilkS")
-		)
-		(fp_line
-			(start -1.4 -4.15)
-			(end -4.25 -1.6)
-			(stroke
-				(width 0.12)
-				(type solid)
-			)
-			(layer "F.SilkS")
-		)
-		(fp_line
-			(start -1.4 4.15)
-			(end 11.45 4.15)
-			(stroke
-				(width 0.12)
-				(type solid)
-			)
-			(layer "F.SilkS")
-		)
-		(fp_line
-			(start 11.45 -4.15)
-			(end -1.4 -4.15)
-			(stroke
-				(width 0.12)
-				(type solid)
-			)
-			(layer "F.SilkS")
-		)
-		(fp_line
-			(start 11.45 4.15)
-			(end 11.45 -4.15)
-			(stroke
-				(width 0.12)
-				(type solid)
-			)
-			(layer "F.SilkS")
-		)
-		(fp_line
-			(start -4.65 -1.85)
-			(end -1.6 -4.6)
-			(stroke
-				(width 0.05)
-				(type solid)
-			)
-			(layer "F.CrtYd")
-		)
-		(fp_line
-			(start -4.65 1.85)
-			(end -4.65 -1.85)
-			(stroke
-				(width 0.05)
-				(type solid)
-			)
-			(layer "F.CrtYd")
-		)
-		(fp_line
-			(start -1.6 -4.6)
-			(end 11.85 -4.6)
-			(stroke
-				(width 0.05)
-				(type solid)
-			)
-			(layer "F.CrtYd")
-		)
-		(fp_line
-			(start -1.6 4.6)
-			(end -4.65 1.85)
-			(stroke
-				(width 0.05)
-				(type solid)
-			)
-			(layer "F.CrtYd")
-		)
-		(fp_line
-			(start 11.85 -4.6)
-			(end 11.85 4.6)
-			(stroke
-				(width 0.05)
-				(type solid)
-			)
-			(layer "F.CrtYd")
-		)
-		(fp_line
-			(start 11.85 4.6)
-			(end -1.6 4.6)
-			(stroke
-				(width 0.05)
-				(type solid)
-			)
-			(layer "F.CrtYd")
-		)
-		(fp_line
-			(start -4.15 -1.55)
-			(end -4.15 1.55)
-			(stroke
-				(width 0.12)
-				(type solid)
-			)
-			(layer "F.Fab")
-		)
-		(fp_line
-			(start -4.15 1.55)
-			(end -1.4 4.05)
-			(stroke
-				(width 0.12)
-				(type solid)
-			)
-			(layer "F.Fab")
-		)
-		(fp_line
-			(start -1.4 -4.05)
-			(end -4.15 -1.55)
-			(stroke
-				(width 0.12)
-				(type solid)
-			)
-			(layer "F.Fab")
-		)
-		(fp_line
-			(start -1.4 4.05)
-			(end 11.35 4.05)
-			(stroke
-				(width 0.12)
-				(type solid)
-			)
-			(layer "F.Fab")
-		)
-		(fp_line
-			(start 11.35 -4.05)
-			(end -1.4 -4.05)
-			(stroke
-				(width 0.12)
-				(type solid)
-			)
-			(layer "F.Fab")
-		)
-		(fp_line
-			(start 11.35 4.05)
-			(end 11.35 -4.05)
-			(stroke
-				(width 0.12)
-				(type solid)
-			)
-			(layer "F.Fab")
-		)
-		(fp_text user "${REFERENCE}"
-			(at 3.6 0.05 0)
-			(layer "F.Fab")
-			(effects
-				(font
-					(size 1 1)
-					(thickness 0.15)
-				)
-			)
-		)
-		(pad "1" thru_hole roundrect
-			(at 0 0)
+			(start -9.75 -8.15)
+			(end -9.75 -5)
+			(stroke
+				(width 0.12)
+				(type solid)
+			)
+			(layer "F.SilkS")
+		)
+		(fp_line
+			(start -9.75 -5)
+			(end -6.9 -2.4)
+			(stroke
+				(width 0.12)
+				(type solid)
+			)
+			(layer "F.SilkS")
+		)
+		(fp_line
+			(start -6.9 -10.7)
+			(end -9.75 -8.15)
+			(stroke
+				(width 0.12)
+				(type solid)
+			)
+			(layer "F.SilkS")
+		)
+		(fp_line
+			(start -6.9 -2.4)
+			(end 5.95 -2.4)
+			(stroke
+				(width 0.12)
+				(type solid)
+			)
+			(layer "F.SilkS")
+		)
+		(fp_line
+			(start 5.95 -10.7)
+			(end -6.9 -10.7)
+			(stroke
+				(width 0.12)
+				(type solid)
+			)
+			(layer "F.SilkS")
+		)
+		(fp_line
+			(start 5.95 -2.4)
+			(end 5.95 -10.7)
+			(stroke
+				(width 0.12)
+				(type solid)
+			)
+			(layer "F.SilkS")
+		)
+		(fp_line
+			(start -10.15 -8.4)
+			(end -7.1 -11.15)
+			(stroke
+				(width 0.05)
+				(type solid)
+			)
+			(layer "F.CrtYd")
+		)
+		(fp_line
+			(start -10.15 -4.7)
+			(end -10.15 -8.4)
+			(stroke
+				(width 0.05)
+				(type solid)
+			)
+			(layer "F.CrtYd")
+		)
+		(fp_line
+			(start -7.1 -11.15)
+			(end 6.35 -11.15)
+			(stroke
+				(width 0.05)
+				(type solid)
+			)
+			(layer "F.CrtYd")
+		)
+		(fp_line
+			(start -7.1 -1.95)
+			(end -10.15 -4.7)
+			(stroke
+				(width 0.05)
+				(type solid)
+			)
+			(layer "F.CrtYd")
+		)
+		(fp_line
+			(start 6.35 -11.15)
+			(end 6.35 -1.95)
+			(stroke
+				(width 0.05)
+				(type solid)
+			)
+			(layer "F.CrtYd")
+		)
+		(fp_line
+			(start 6.35 -1.95)
+			(end -7.1 -1.95)
+			(stroke
+				(width 0.05)
+				(type solid)
+			)
+			(layer "F.CrtYd")
+		)
+		(fp_line
+			(start -9.65 -8.1)
+			(end -9.65 -5)
+			(stroke
+				(width 0.12)
+				(type solid)
+			)
+			(layer "F.Fab")
+		)
+		(fp_line
+			(start -9.65 -5)
+			(end -6.9 -2.5)
+			(stroke
+				(width 0.12)
+				(type solid)
+			)
+			(layer "F.Fab")
+		)
+		(fp_line
+			(start -6.9 -10.6)
+			(end -9.65 -8.1)
+			(stroke
+				(width 0.12)
+				(type solid)
+			)
+			(layer "F.Fab")
+		)
+		(fp_line
+			(start -6.9 -2.5)
+			(end 5.85 -2.5)
+			(stroke
+				(width 0.12)
+				(type solid)
+			)
+			(layer "F.Fab")
+		)
+		(fp_line
+			(start 5.85 -10.6)
+			(end -6.9 -10.6)
+			(stroke
+				(width 0.12)
+				(type solid)
+			)
+			(layer "F.Fab")
+		)
+		(fp_line
+			(start 5.85 -2.5)
+			(end 5.85 -10.6)
+			(stroke
+				(width 0.12)
+				(type solid)
+			)
+			(layer "F.Fab")
+		)
+		(fp_text user "-"
+			(at -6.43 -11.07 0)
+			(unlocked yes)
+			(layer "F.SilkS")
+			(effects
+				(font
+					(size 1 1)
+					(thickness 0.1)
+				)
+				(justify left bottom)
+			)
+		)
+		(fp_text user "+"
+			(at 1.23 -11.3 0)
+			(unlocked yes)
+			(layer "F.SilkS")
+			(effects
+				(font
+					(size 1 1)
+					(thickness 0.1)
+				)
+				(justify left bottom)
+			)
+		)
+		(pad "1" thru_hole circle
+			(at 1.7 -6.55)
+			(size 6 6)
+			(drill 4.5)
+			(layers "*.Cu" "*.Mask")
+			(remove_unused_layers no)
+			(net 2 "V_SW")
+			(pinfunction "+")
+			(pintype "passive")
+		)
+		(pad "2" thru_hole roundrect
+			(at -5.5 -6.55)
 			(size 6 6)
 			(drill 4.5)
@@
 			(remove_unused_layers no)
 			(roundrect_rratio 0.25)
-			(net 2 "V_SW")
-			(pinfunction "+")
-			(pintype "passive")
-		)
-		(pad "2" thru_hole circle
-			(at 7.2 0)
-			(size 6 6)
-			(drill 4.5)
-			(layers "*.Cu" "*.Mask")
-			(remove_unused_layers no)
 			(net 1 "C_GND")
 			(pinfunction "-")
 			(pintype "passive")
 		)
-		(model "${KICAD8_3DMODEL_DIR}/Connector_AMASS.3dshapes/AMASS_XT60-M_1x02_P7.2mm_Vertical.wrl"
-			(offset
-				(xyz 0 0 0)
-			)
-			(scale
-				(xyz 1 1 1)
-			)
-			(rotate
-				(xyz 0 0 0)
-			)
-		)
 	)

Commit message: Update line_f.kicad_pcb
Parts:
- moved MPU1 2.74 mm to (83.2, 163.8)

Commit message: 4#
Parts:
- removed LSA_ANALOG1: ~, LINE_F_FOOT_LIB:LSA_ANALOG
- moved BUCK1 49.9 mm to (94.6, 116.3), turned to 90 degrees
- moved m1 0.26 mm to (90.6, 72.5)
Connections:
- LSA_UART1 pad 4: unconnected-(LSA_UART1-AN-Pad4) -> LSA_AN
- m1 pad 10: AI2 -> D3
- m1 pad 11: AI1 -> D4
- m1 pad 12: BI1 -> D5
- m1 pad 13: BI2 -> unconnected-(m1-B5-Pad13)
- m1 pad 17: unconnected-(m1-B9-Pad17) -> D0
- m1 pad 26: D5 -> D2
- m1 pad 27: D4 -> D1
- m1 pad 28: D3 -> LSA_AN
- m1 pad 29: D2 -> BI2
- m1 pad 30: D1 -> BI1
- m1 pad 31: D0 -> AI1
- m1 pad 32: LSA_AN -> AI2
- m1 pad 33: unconnected-(m1-A2-Pad33) -> PWMB
- m1 pad 34: PWMB -> PWMA
- m1 pad 35: PWMA -> unconnected-(m1-A0-Pad35)

Commit message: 4#
Parts:
- moved LSA_UART1 75.9 mm to (60.7, 138.1)
- moved D1 28.2 mm to (59.9, 167.8)
- moved M3 23.5 mm to (57.5, 146.4)
- moved U1 23.3 mm to (132.4, 127.8)
- moved M2 22.8 mm to (127.5, 146.2)
- moved LSA_DIGITAL1 10.5 mm to (63.1, 122.6)
- moved SW1 8.01 mm to (31.0, 125.7)
- moved SW3 1.91 mm to (124.0, 174.6)
- moved SW4 1.91 mm to (141.0, 174.7)
Other:
- outline, holes or cut-outs redrawn
- board text removed: "Run"
- board text removed: "Run2'"
Changed lines of the file:
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@@
 	(footprint "LINE_F_FOOT_LIB:LED_LINE"
 		(layer "F.Cu")
-		(at 31.95 171.31)
+		(at 59.91 167.81)
 		(property "Reference" "D1"
 			(at -3 -6 0)
@@
 	(footprint "LINE_F_FOOT_LIB:LSA_UART"
 		(layer "F.Cu")
-		(at 136.2 129.59)
+		(at 60.74 138.09)
 		(property "Reference" "LSA_UART1"
 			(at 1.2625 -0.91 0)
@@
 	(footprint "LINE_F_FOOT_LIB:connector_motor"
 		(layer "F.Cu")
-		(at 149.48 152.18 90)
+		(at 127.48 146.18 90)
 		(property "Reference" "M2"
 			(at 0 -0.5 90)
@@
 	(footprint "LINE_F_FOOT_LIB:push_button"
 		(layer "F.Cu")
-		(at 124 176.5 90)
+		(at 123.952 174.588 90)
 		(property "Reference" "SW3"
 			(at 0.762 -3.302 90)
@@
 	(footprint "LINE_F_FOOT_LIB:battery_sw"
 		(layer "F.Cu")
-		(at 35.5 132.315 -90)
+		(at 31 125.685 -90)
 		(property "Reference" "SW1"
 			(at 0.06 5.17 90)
@@
 	(footprint "LINE_F_FOOT_LIB:push_button"
 		(layer "F.Cu")
-		(at 141.032 176.588 90)
+		(at 140.984 174.676 90)
 		(property "Reference" "SW4"
 			(at 0.762 -3.302 90)
@@
 	(footprint "LINE_F_FOOT_LIB:LSA_DIGITAL"
 		(layer "F.Cu")
-		(at 72.6 127.11)
+		(at 63.1 122.61)
 		(property "Reference" "LSA_DIGITAL1"
 			(at 0 -0.5 0)
@@
 	(footprint "LINE_F_FOOT_LIB:TB6612FNG_LINE"
 		(layer "F.Cu")
-		(at 126.38 150.31)
+		(at 132.38 127.81)
 		(property "Reference" "U1"
 			(at 0.17 -8.12 0)
@@
 	(footprint "LINE_F_FOOT_LIB:connector_motor"
 		(layer "F.Cu")
-		(at 34.52 151.32 -90)
+		(at 57.52 146.36 -90)
 		(property "Reference" "M3"
 			(at 0 -0.5 -90)
@@
 	(gr_poly
 		(pts
-			(xy 25.5 186) (xy 160 186) (xy 160 114) (xy 114 114) (xy 114 43.5) (xy 161.5 43.5) (xy 161.5 26.5)
+			(xy 26.5 183.5) (xy 161 183.5) (xy 160 114) (xy 114 114) (xy 114 43.5) (xy 161.5 43.5) (xy 161.5 26.5)
 			(xy 24 26.5) (xy 24 44) (xy 68 44) (xy 68 115) (xy 25.5 115) (xy 25.5 186)
 		)
@@
 	)
 	(gr_circle
-		(center 152 152.5)
-		(end 154 152.5)
-		(stroke
-			(width 0.05)
-			(type default)
-		)
-		(fill none)
-		(layer "Edge.Cuts")
-	)
-	(gr_circle
-		(center 155.5 161)
-		(end 156.262 161.762)
+		(center 151.93837 161.01)
+		(end 152.70037 161.772)
 		(stroke
 			(width 0.05)
@@
 	)
 	(gr_circle
-		(center 32.5 151)
-		(end 34.5 151)
-		(stroke
-			(width 0.05)
-			(type default)
-		)
-		(fill none)
-		(layer "Edge.Cuts")
-	)
-	(gr_circle
-		(center 29.016 159.51)
-		(end 29.778 160.272)
+		(center 33.43837 159.51)
+		(end 34.20037 160.272)
 		(stroke
 			(width 0.05)
@@
 	)
 	(gr_circle
-		(center 29.07763 143)
-		(end 29.83963 143.762)
+		(center 152 144.5)
+		(end 152.762 145.262)
 		(stroke
 			(width 0.05)
@@
 	)
 	(gr_circle
-		(center 155.56163 144.49)
-		(end 156.32363 145.252)
+		(center 33.5 143)
+		(end 34.262 143.762)
 		(stroke
 			(width 0.05)
@@
 		(layer "Edge.Cuts")
 	)
-	(gr_text "Run"
-		(at 154 183.5 0)
-		(layer "F.Cu")
-		(effects
-			(font
-				(size 1.5 1.5)
-				(thickness 0.3)
-				(bold yes)
-			)
-			(justify left bottom)
-		)
-	)
 	(gr_text "BTZ"
-		(at 140 184 0)
+		(at 144.5 182.5 0)
 		(layer "F.SilkS")
 		(effects
@@
 		)
 	)
-	(gr_text "Run2'"
-		(at 154.5 180 0)
-		(layer "F.Mask")
-		(effects
-			(font
-				(size 1 1)
-				(thickness 0.15)
+	(dimension
+		(type aligned)
+		(layer "F.Cu")
+		(pts
+			(xy 48.5 151) (xy 25.5 151)
+		)
+		(height 0)
+		(gr_text "23.0000 mm"
+			(at 37 149.2 0)
+			(layer "F.Cu")
+			(effects
+				(font
+					(size 1.5 1.5)
+					(thickness 0.3)
+				)
 			)
-			(justify left bottom)
 		)
+		(format
+			(prefix "")
+			(suffix "")
+			(units 3)
+			(units_format 1)
+			(precision 4)
+		)
+		(style
+			(thickness 0.2)
+			(arrow_length 1.27)
+			(text_position_mode 0)
+			(extension_height 0.58642)
+			(extension_offset 0.5) keep_text_aligned)
+	)
+	(dimension
+		(type aligned)
+		(layer "F.Cu")
+		(pts
+			(xy 160 152) (xy 137 152)
+		)
+		(height 0)
+		(gr_text "23.0000 mm"
+			(at 148.5 150.2 0)
+			(layer "F.Cu")
+			(effects
+				(font
+					(size 1.5 1.5)
+					(thickness 0.3)
+				)
+			)
+		)
+		(format
+			(prefix "")
+			(suffix "")
+			(units 3)
+			(units_format 1)
+			(precision 4)
+		)
+		(style
+			(thickness 0.2)
+			(arrow_length 1.27)
+			(text_position_mode 0)
+			(extension_height 0.58642)
+			(extension_offset 0.5) keep_text_aligned)
 	)
 	(group ""

Commit message: 4#
Parts:
- moved BT1 167.0 mm to (-74.0, 109.2)
- moved BUCK1 167.0 mm to (-72.4, 113.0)
- moved D1 167.0 mm to (-107.1, 164.5)
- moved LSA_DIGITAL1 167.0 mm to (-103.9, 119.3)
- moved LSA_UART1 167.0 mm to (-106.3, 134.8)
- moved M2 167.0 mm to (-39.5, 142.9)
- moved M3 167.0 mm to (-109.5, 143.0)
- moved MPU1 167.0 mm to (-83.8, 160.5)
- moved R1 167.0 mm to (-109.2, 174.0)
- moved SW1 167.0 mm to (-136.0, 122.4)
- moved SW2 167.0 mm to (-132.5, 176.2)
- moved SW3 167.0 mm to (-43.0, 171.3)
- moved SW4 167.0 mm to (-26.0, 171.4)
- moved U1 167.0 mm to (-34.6, 124.5)
- moved m1 167.0 mm to (-76.4, 69.2)
Other:
- board size 137.5 x 159.5 mm -> 137.5 x 157 mm

Commit message: 4#
Parts:
- moved R1 4.52 mm to (-107.3, 169.9)
- moved SW2 4.52 mm to (-130.6, 172.1)
- moved SW3 2.73 mm to (-43.5, 168.6)
- moved SW4 2.73 mm to (-26.5, 168.7)
Other:
- outline, holes or cut-outs redrawn
Changed lines of the file:
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@@
 	(footprint "LINE_F_FOOT_LIB:push_button"
 		(layer "F.Cu")
-		(at -43.048 171.268 90)
+		(at -43.548 168.588 90)
 		(property "Reference" "SW3"
 			(at 0.762 -3.302 90)
@@
 	(footprint "LINE_F_FOOT_LIB:push_button"
 		(layer "F.Cu")
-		(at -26.016 171.356 90)
+		(at -26.516 168.676 90)
 		(property "Reference" "SW4"
 			(at 0.762 -3.302 90)
@@
 	(footprint "LINE_F_FOOT_LIB:SLIDE SW"
 		(layer "F.Cu")
-		(at -132.5 176.18)
+		(at -130.59 172.08)
 		(property "Reference" "SW2"
 			(at -6.94 -3.79 0)
@@
 	(footprint "LINE_F_FOOT_LIB:RESISTOR_LINE"
 		(layer "F.Cu")
-		(at -109.17 174.03)
+		(at -107.26 169.93)
 		(property "Reference" "R1"
 			(at 0 -0.5 0)
@@
 	)
 	(gr_rect
-		(start -92 111.5)
-		(end -60 171.5)
+		(start -92 115.5)
+		(end -60 175.5)
 		(stroke
 			(width 0.1)
@@
 	)
 	(gr_line
-		(start -141.5 180)
-		(end -9.043476 180.18)
+		(start -136.5 177.5)
+		(end -9.043476 177.179999)
 		(stroke
 			(width 0.05)
@@
 	)
 	(gr_text "BTZ"
-		(at -22.5 179.18 0)
+		(at -18.5 172 0)
 		(layer "F.SilkS")
 		(effects
