File: Line_kicad/line_f/line_f.kicad_pcb (KiCad board)
At the start: 2 copper layers, 137.5 x 154 mm, 15 parts, among them M2 Motor_DC, M3 Motor_DC, SW1 SW_SPST, SW2 SW_SPDT, SW3 SW_Push, SW4 SW_Push, U1 TB6612FNG_LINE, m1 BLACKPILL

Commit message: v9.0
Parts:
- moved m1 0.51 mm to (-75.9, 69.1)

Commit message: 6updatefrmsch#
Connections:
- LSA_UART1 pad 4: LSA_AN -> unconnected-(LSA_UART1-AN-Pad4)
- m1 pad 10: D3 -> LSA_UEN
- m1 pad 11: D4 -> PRIORITY_SW
- m1 pad 12: D5 -> JPULSE
- m1 pad 13: unconnected-(m1-B5-Pad13) -> SW_RUN
- m1 pad 16: D6 -> AI1
- m1 pad 17: D0 -> AI2
- m1 pad 19: unconnected-(m1-GND-Pad19) -> C_GND
- m1 pad 2: SW_RUN -> D3
- m1 pad 22: C_GND -> unconnected-(m1-GND-Pad22)
- m1 pad 26: D2 -> D6
- m1 pad 27: D1 -> D5
- m1 pad 28: LSA_AN -> D4
- m1 pad 29: BI2 -> PWMB
- m1 pad 3: LED_F -> D2
- m1 pad 30: BI1 -> BI2
- m1 pad 31: AI1 -> BI1
- m1 pad 32: AI2 -> LSA_TX
- m1 pad 33: PWMB -> LSA_RX
- m1 pad 4: SW_TRY -> D1
- m1 pad 5: JPULSE -> D0
- m1 pad 6: LSA_RX -> unconnected-(m1-A9-Pad6)
- m1 pad 7: LSA_TX -> unconnected-(m1-A10-Pad7)
- m1 pad 8: LSA_UEN -> SW_TRY
- m1 pad 9: PRIORITY_SW -> LED_F
Changed lines of the file:
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@@
 	(net 4 "5V")
 	(net 5 "Net-(D1-A)")
-	(net 6 "LSA_AN")
+	(net 6 "unconnected-(LSA_UART1-AN-Pad4)")
 	(net 7 "JPULSE")
 	(net 8 "D7")
@@
 	(net 15 "D2")
 	(net 16 "LSA_UEN")
-	(net 17 "unconnected-(m1-B5-Pad13)")
+	(net 17 "unconnected-(m1-A9-Pad6)")
 	(net 18 "unconnected-(LSA_UART1-Orphan-Pad8)")
 	(net 19 "unconnected-(LSA_UART1-Orphan1-Pad6)")
@@
 	(net 27 "unconnected-(m1-A0-Pad35)")
 	(net 28 "unconnected-(m1-C13-Pad39)")
-	(net 29 "unconnected-(m1-GND-Pad19)")
+	(net 29 "unconnected-(m1-GND-Pad22)")
 	(net 30 "BI1")
 	(net 31 "PWMA")
@@
 	(net 55 "unconnected-(U1-GND-Pad8)")
 	(net 56 "unconnected-(U1-GND-Pad3)")
+	(net 57 "unconnected-(m1-A10-Pad7)")
 	(footprint "LINE_F_FOOT_LIB:BATTERY_LINE_XT60"
 		(layer "F.Cu")
@@
 			)
 		)
-		(sheetname "Root")
+		(sheetname "/")
 		(sheetfile "line_f.kicad_sch")
 		(attr through_hole)
@@
 			)
 		)
-		(sheetname "Root")
+		(sheetname "/")
 		(sheetfile "line_f.kicad_sch")
 		(attr smd)
@@
 			)
 		)
-		(sheetname "Root")
+		(sheetname "/")
 		(sheetfile "line_f.kicad_sch")
 		(attr through_hole)
@@
 			)
 		)
+		(property "Sim.Pins" "1=K 2=A"
+			(at 0 0 0)
+			(unlocked yes)
+			(layer "F.Fab")
+			(hide yes)
+			(effects
+				(font
+					(size 1 1)
+					(thickness 0.15)
+				)
+			)
+		)
 		(property ki_fp_filters "LED* LED_SMD:* LED_THT:*")
-		(sheetname "Root")
+		(sheetname "/")
 		(sheetfile "line_f.kicad_sch")
 		(attr through_hole)
@@
 			)
 		)
-		(sheetname "Root")
+		(sheetname "/")
 		(sheetfile "line_f.kicad_sch")
 		(fp_line
@@
 			(layers "*.Cu" "*.Mask")
 			(remove_unused_layers no)
-			(net 44 "SW_RUN")
+			(net 13 "D3")
 			(pinfunction "B13")
 			(pintype "bidirectional")
@@
 			(layers "*.Cu" "*.Mask")
 			(remove_unused_layers no)
-			(net 42 "LED_F")
+			(net 15 "D2")
 			(pinfunction "B14")
 			(pintype "bidirectional")
@@
 			(layers "*.Cu" "*.Mask")
 			(remove_unused_layers no)
-			(net 41 "SW_TRY")
+			(net 12 "D1")
 			(pinfunction "B15")
 			(pintype "bidirectional")
@@
 			(layers "*.Cu" "*.Mask")
 			(remove_unused_layers no)
-			(net 7 "JPULSE")
+			(net 11 "D0")
 			(pinfunction "A8")
 			(pintype "bidirectional")
@@
 			(layers "*.Cu" "*.Mask")
 			(remove_unused_layers no)
-			(net 20 "LSA_RX")
+			(net 17 "unconnected-(m1-A9-Pad6)")
 			(pinfunction "A9")
-			(pintype "bidirectional")
+			(pintype "bidirectional+no_connect")
 			(solder_mask_margin 0.0508)
 			(thermal_bridge_angle 0)
@@
 			(layers "*.Cu" "*.Mask")
 			(remove_unused_layers no)
-			(net 22 "LSA_TX")
+			(net 57 "unconnected-(m1-A10-Pad7)")
 			(pinfunction "A10")
-			(pintype "bidirectional")
+			(pintype "bidirectional+no_connect")
 			(solder_mask_margin 0.0508)
 			(thermal_bridge_angle 0)
@@
 			(layers "*.Cu" "*.Mask")
 			(remove_unused_layers no)
-			(net 16 "LSA_UEN")
+			(net 41 "SW_TRY")
 			(pinfunction "A11")
 			(pintype "bidirectional")
@@
 			(layers "*.Cu" "*.Mask")
 			(remove_unused_layers no)
-			(net 23 "PRIORITY_SW")
+			(net 42 "LED_F")
 			(pinfunction "A12")
 			(pintype "bidirectional")
@@
 			(layers "*.Cu" "*.Mask")
 			(remove_unused_layers no)
-			(net 13 "D3")
+			(net 16 "LSA_UEN")
 			(pinfunction "A15")
 			(pintype "bidirectional")
@@
 			(layers "*.Cu" "*.Mask")
 			(remove_unused_layers no)
-			(net 10 "D4")
+			(net 23 "PRIORITY_SW")
 			(pinfunction "B3")
 			(pintype "bidirectional")
@@
 			(layers "*.Cu" "*.Mask")
 			(remove_unused_layers no)
-			(net 14 "D5")
+			(net 7 "JPULSE")
 			(pinfunction "B4")
 			(pintype "bidirectional")
@@
 			(layers "*.Cu" "*.Mask")
 			(remove_unused_layers no)
-			(net 17 "unconnected-(m1-B5-Pad13)")
+			(net 44 "SW_RUN")
 			(pinfunction "B5")
-			(pintype "no_connect")
+			(pintype "bidirectional")
 			(solder_mask_margin 0.0508)
 			(thermal_bridge_angle 0)
@@
 			(layers "*.Cu" "*.Mask")
 			(remove_unused_layers no)
-			(net 9 "D6")
+			(net 37 "AI1")
 			(pinfunction "B8")
 			(pintype "bidirectional")
@@
 			(layers "*.Cu" "*.Mask")
 			(remove_unused_layers no)
-			(net 11 "D0")
+			(net 38 "AI2")
 			(pinfunction "B9")
 			(pintype "bidirectional")
@@
 			(layers "*.Cu" "*.Mask")
 			(remove_unused_layers no)
-			(net 29 "unconnected-(m1-GND-Pad19)")
+			(net 1 "C_GND")
 			(pinfunction "GND")
-			(pintype "power_in+no_connect")
+			(pintype "power_in")
 			(solder_mask_margin 0.0508)
 			(thermal_bridge_angle 0)
@@
 			(layers "*.Cu" "*.Mask")
 			(remove_unused_layers no)
-			(net 1 "C_GND")
+			(net 29 "unconnected-(m1-GND-Pad22)")
 			(pinfunction "GND")
-			(pintype "power_in")
+			(pintype "power_in+no_connect")
 			(solder_mask_margin 0.0508)
 			(thermal_bridge_angle 0)
@@
 			(layers "*.Cu" "*.Mask")
 			(remove_unused_layers no)
-			(net 15 "D2")
+			(net 9 "D6")
 			(pinfunction "B1")
 			(pintype "bidirectional")
@@
 			(layers "*.Cu" "*.Mask")
 			(remove_unused_layers no)
-			(net 12 "D1")
+			(net 14 "D5")
 			(pinfunction "B0")
 			(pintype "bidirectional")
@@
 			(layers "*.Cu" "*.Mask")
 			(remove_unused_layers no)
-			(net 6 "LSA_AN")
+			(net 10 "D4")
 			(pinfunction "A7")
 			(pintype "bidirectional")
@@
 			(layers "*.Cu" "*.Mask")
 			(remove_unused_layers no)
-			(net 26 "BI2")
+			(net 33 "PWMB")
 			(pinfunction "A6")
 			(pintype "bidirectional")
@@
 			(layers "*.Cu" "*.Mask")
 			(remove_unused_layers no)
-			(net 30 "BI1")
+			(net 26 "BI2")
 			(pinfunction "A5")
 			(pintype "bidirectional")
@@
 			(layers "*.Cu" "*.Mask")
 			(remove_unused_layers no)
-			(net 37 "AI1")
+			(net 30 "BI1")
 			(pinfunction "A4")
 			(pintype "bidirectional")
@@
 			(layers "*.Cu" "*.Mask")
 			(remove_unused_layers no)
-			(net 38 "AI2")
+			(net 22 "LSA_TX")
 			(pinfunction "A3")
 			(pintype "bidirectional")
@@
 			(layers "*.Cu" "*.Mask")
 			(remove_unused_layers no)
-			(net 33 "PWMB")
+			(net 20 "LSA_RX")
 			(pinfunction "A2")
 			(pintype "bidirectional")
@@
 			(net 27 "unconnected-(m1-A0-Pad35)")
 			(pinfunction "A0")
-			(pintype "no_connect")
+			(pintype "bidirectional+no_connect")
 			(solder_mask_margin 0.0508)
 			(thermal_bridge_angle 0)
@@
 			)
 		)
-		(sheetname "Root")
+		(sheetname "/")
 		(sheetfile "line_f.kicad_sch")
 		(attr through_hole)
@@
 			(layers "*.Cu" "*.Mask")
 			(remove_unused_layers no)
-			(net 6 "LSA_AN")
+			(net 6 "unconnected-(LSA_UART1-AN-Pad4)")
 			(pinfunction "AN")
-			(pintype "bidirectional")
+			(pintype "bidirectional+no_connect")
 		)
 		(pad "5" thru_hole circle
@@
 		)
 		(property ki_fp_filters "PinHeader*P2.54mm* TerminalBlock*")
-		(sheetname "Root")
+		(sheetname "/")
 		(sheetfile "line_f.kicad_sch")
 		(attr through_hole)
@@
 			)
 		)
-		(sheetname "Root")
+		(sheetname "/")
 		(sheetfile "line_f.kicad_sch")
 		(attr through_hole)
@@
 			)
 		)
-		(sheetname "Root")
+		(sheetname "/")
 		(sheetfile "line_f.kicad_sch")
 		(fp_rect
@@
 			)
 		)
-		(sheetname "Root")
+		(sheetname "/")
 		(sheetfile "line_f.kicad_sch")
 		(attr through_hole)
@@
 			)
 		)
-		(sheetname "Root")
+		(sheetname "/")
 		(sheetfile "line_f.kicad_sch")
 		(attr through_hole)
@@
 			)
 		)
-		(sheetname "Root")
+		(sheetname "/")
 		(sheetfile "line_f.kicad_sch")
 		(attr through_hole)
@@
 			)
 		)
-		(sheetname "Root")
+		(sheetname "/")
 		(sheetfile "line_f.kicad_sch")
 		(attr through_hole)
@@
 		)
 		(property ki_fp_filters "R_*")
-		(sheetname "Root")
+		(sheetname "/")
 		(sheetfile "line_f.kicad_sch")
 		(attr through_hole)
@@
 		)
 		(property ki_fp_filters "PinHeader*P2.54mm* TerminalBlock*")
-		(sheetname "Root")
+		(sheetname "/")
 		(sheetfile "line_f.kicad_sch")
 		(attr through_hole)

Commit message: 6halfshape#
Other:
- board size 137.5 x 154 mm -> 235.5 x 156.1 mm
Changed lines of the file:
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@@
 		(layer "F.SilkS")
+	)
+	(gr_line
+		(start 25 21)
+		(end 92.5 21)
+		(stroke
+			(width 0.05)
+			(type default)
+		)
+		(layer "Edge.Cuts")
 	)
 	(gr_arc
@@
 	)
 	(gr_line
+		(start 25 111)
+		(end 25 171)
+		(stroke
+			(width 0.05)
+			(type default)
+		)
+		(layer "Edge.Cuts")
+	)
+	(gr_line
 		(start -138.503031 177.003028)
 		(end -9.090337 177.133761)
@@
 		(layer "Edge.Cuts")
 	)
+	(gr_line
+		(start 25 41)
+		(end 25 21)
+		(stroke
+			(width 0.05)
+			(type default)
+		)
+		(layer "Edge.Cuts")
+	)
 	(gr_circle
 		(center -15.06163 157.69)
@@
 		)
 		(fill no)
+		(layer "Edge.Cuts")
+	)
+	(gr_line
+		(start 25 171)
+		(end 92.5 171)
+		(stroke
+			(width 0.05)
+			(type default)
+		)
 		(layer "Edge.Cuts")
 	)
@@
 		(layer "Edge.Cuts")
 	)
+	(gr_line
+		(start 25 111)
+		(end 72.5 111)
+		(stroke
+			(width 0.05)
+			(type solid)
+		)
+		(layer "Edge.Cuts")
+	)
+	(gr_line
+		(start 25 41)
+		(end 72.5 41)
+		(stroke
+			(width 0.05)
+			(type solid)
+		)
+		(layer "Edge.Cuts")
+	)
 	(gr_circle
 		(center -76.5 49.18)
@@
 		)
 		(fill no)
+		(layer "Edge.Cuts")
+	)
+	(gr_line
+		(start 72.5 111)
+		(end 72.5 41)
+		(stroke
+			(width 0.05)
+			(type solid)
+		)
 		(layer "Edge.Cuts")
 	)
@@
 	)
 	(dimension
-		(type aligned)
-		(layer "F.Cu")
+		(type orthogonal)
+		(layer "F.SilkS")
 		(pts
-			(xy -118.5 147.68) (xy -141.5 147.68)
-		)
-		(height 0)
+			(xy -6.522537 149.5) (xy -26.5 150)
+		)
+		(height 0.5)
+		(orientation 0)
 		(format
 			(prefix "")
@@
 		)
 		(style
-			(thickness 0.2)
+			(thickness 0.1)
 			(arrow_length 1.27)
 			(text_position_mode 0)
@@
 			(keep_text_aligned yes)
 		)
-		(gr_text "23.0000 mm"
-			(at -130 145.88 0)
-			(layer "F.Cu")
+		(gr_text "19.9775 mm"
+			(at -16.511269 148.9 0)
+			(layer "F.SilkS")
 			(effects
 				(font
-					(size 1.5 1.5)
-					(thickness 0.3)
+					(size 1 1)
+					(thickness 0.1)
 				)
 			)
@@
 	)
 	(dimension
-		(type aligned)
-		(layer "F.Cu")
+		(type orthogonal)
+		(layer "F.SilkS")
 		(pts
-			(xy -7 148.68) (xy -30 148.68)
-		)
-		(height 0)
+			(xy -121.522537 147.5) (xy -141.5 148)
+		)
+		(height 0.5)
+		(orientation 0)
 		(format
 			(prefix "")
@@
 		)
 		(style
-			(thickness 0.2)
+			(thickness 0.1)
 			(arrow_length 1.27)
 			(text_position_mode 0)
@@
 			(keep_text_aligned yes)
 		)
-		(gr_text "23.0000 mm"
-			(at -18.5 146.88 0)
-			(layer "F.Cu")
+		(gr_text "19.9775 mm"
+			(at -131.511269 146.9 0)
+			(layer "F.SilkS")
 			(effects
 				(font
-					(size 1.5 1.5)
-					(thickness 0.3)
+					(size 1 1)
+					(thickness 0.1)
 				)
 			)
+		)
+	)
+	(dimension
+		(type orthogonal)
+		(layer "Edge.Cuts")
+		(pts
+			(xy -95 41) (xy -95 111)
+		)
+		(height -53)
+		(orientation 1)
+		(format
+			(prefix "")
+			(suffix "")
+			(units 3)
+			(units_format 1)
+			(precision 4)
+		)
+		(style
+			(thickness 0.05)
+			(arrow_length 1.27)
+			(text_position_mode 0)
+			(arrow_direction outward)
+			(extension_height 0.58642)
+			(extension_offset 0.5)
+			(keep_text_aligned yes)
+		)
+		(gr_text "70.0000 mm"
+			(at -149.15 76 90)
+			(layer "Edge.Cuts")
+			(effects
+				(font
+					(size 1 1)
+					(thickness 0.15)
+				)
+			)

Commit message: 6baseshape#
Other:
- board size 235.5 x 156.1 mm -> 298 x 155.1 mm
Changed lines of the file:
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@@
 	)
 	(gr_line
-		(start 25 21)
-		(end 92.5 21)
+		(start 155 22)
+		(end 87.5 22)
+		(stroke
+			(width 0.05)
+			(type default)
+		)
+		(layer "Edge.Cuts")
+	)
+	(gr_line
+		(start 20 42)
+		(end 20 22)
 		(stroke
 			(width 0.05)
@@
 	)
 	(gr_line
+		(start 20 22)
+		(end 87.5 22)
+		(stroke
+			(width 0.05)
+			(type default)
+		)
+		(layer "Edge.Cuts")
+	)
+	(gr_line
 		(start -6.087617 174.090602)
 		(end -6.957456 113.636839)
+		(stroke
+			(width 0.05)
+			(type default)
+		)
+		(layer "Edge.Cuts")
+	)
+	(gr_line
+		(start 20 112)
+		(end 20 172)
 		(stroke
 			(width 0.05)
@@
 	)
 	(gr_line
-		(start 25 111)
-		(end 25 171)
-		(stroke
-			(width 0.05)
-			(type default)
+		(start 155 112)
+		(end 155 172)
+		(stroke
+			(width 0.05)
+			(type default)
+		)
+		(layer "Edge.Cuts")
+	)
+	(gr_line
+		(start 20 112)
+		(end 67.5 112)
+		(stroke
+			(width 0.05)
+			(type solid)
 		)
 		(layer "Edge.Cuts")
@@
 	)
 	(gr_line
-		(start 25 41)
-		(end 25 21)
+		(start 155 42)
+		(end 155 22)
+		(stroke
+			(width 0.05)
+			(type default)
+		)
+		(layer "Edge.Cuts")
+	)
+	(gr_line
+		(start 20 172)
+		(end 87.5 172)
 		(stroke
 			(width 0.05)
@@
 	)
 	(gr_line
-		(start 25 171)
-		(end 92.5 171)
+		(start 155 172)
+		(end 87.5 172)
 		(stroke
 			(width 0.05)
@@
 	)
 	(gr_line
-		(start 25 111)
-		(end 72.5 111)
+		(start 155 112)
+		(end 107.5 112)
 		(stroke
 			(width 0.05)
@@
 	)
 	(gr_line
-		(start 25 41)
-		(end 72.5 41)
+		(start 155 42)
+		(end 107.5 42)
 		(stroke
 			(width 0.05)
@@
 	)
 	(gr_line
-		(start 72.5 111)
-		(end 72.5 41)
+		(start 107.5 112)
+		(end 107.5 42)
 		(stroke
 			(width 0.05)
@@
 			(width 0.05)
 			(type default)
+		)
+		(layer "Edge.Cuts")
+	)
+	(gr_line
+		(start 67.5 112)
+		(end 67.5 42)
+		(stroke
+			(width 0.05)
+			(type solid)
+		)
+		(layer "Edge.Cuts")
+	)
+	(gr_line
+		(start 20 42)
+		(end 67.5 42)
+		(stroke
+			(width 0.05)
+			(type solid)
 		)
 		(layer "Edge.Cuts")
@@
 		(members "2b246de5-1c3e-4b08-8844-68d2926f8eae")
 	)
+	(group ""
+		(members "08e62b6e-ce53-40d2-b3f8-55d689e35f33" "66c1f79e-09a2-49f6-90df-8659d6d0da7c"
+			"b0ed438f-358f-44be-bb09-ac3e2ab8c9ff" "b51dc32d-5a38-49bd-95bd-c49b440edd10"
+		)
+	)
 	(embedded_fonts no)

Commit message: 6baseshape#
Parts:
- moved BT1 7.50 mm to (-81.5, 109.0)
- moved m1 7.50 mm to (-83.4, 68.9)
Other:
- outline, holes or cut-outs redrawn
Changed lines of the file:
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@@
 	(footprint "LINE_F_FOOT_LIB:BATTERY_LINE_XT60"
 		(layer "F.Cu")
-		(at -74 109.23)
+		(at -81.5 109.05)
 		(property "Reference" "BT1"
 			(at 0 -0.5 0)
@@
 	(footprint "LINE_F_FOOT_LIB:FINAL_BLACKPILL_LINE"
 		(layer "F.Cu")
-		(at -75.88 69.07)
+		(at -83.38 68.89)
 		(property "Reference" "m1"
 			(at -0.04 -23.9 0)
@@
 			(type default)
 		)
+		(locked yes)
 		(layer "Edge.Cuts")
 	)
@@
 			(type default)
 		)
+		(locked yes)
 		(layer "Edge.Cuts")
 	)
@@
 			(type default)
 		)
+		(locked yes)
 		(layer "Edge.Cuts")
 	)
@@
 			(type default)
 		)
+		(locked yes)
 		(layer "Edge.Cuts")
 	)
@@
 			(type default)
 		)
+		(locked yes)
 		(layer "Edge.Cuts")
 	)
@@
 			(type solid)
 		)
+		(locked yes)
 		(layer "Edge.Cuts")
 	)
@@
 			(type default)
 		)
+		(locked yes)
 		(layer "Edge.Cuts")
 	)
@@
 			(type default)
 		)
+		(locked yes)
 		(layer "Edge.Cuts")
 	)
@@
 			(type default)
 		)
+		(locked yes)
 		(layer "Edge.Cuts")
 	)
@@
 	)
 	(gr_circle
-		(center -76.5 64.42)
-		(end -74.976 63.658)
+		(center -84 64.24)
+		(end -82.476 63.478)
 		(stroke
 			(width 0.05)
@@
 			(type solid)
 		)
+		(locked yes)
 		(layer "Edge.Cuts")
 	)
@@
 			(type solid)
 		)
+		(locked yes)
 		(layer "Edge.Cuts")
 	)
 	(gr_circle
-		(center -76.5 49.18)
-		(end -74.976 48.418)
+		(center -84 49)
+		(end -82.476 48.238)
 		(stroke
 			(width 0.05)
@@
 			(type solid)
 		)
+		(locked yes)
 		(layer "Edge.Cuts")
 	)
@@
 			(type solid)
 		)
+		(locked yes)
 		(layer "Edge.Cuts")
 	)
@@
 			(type solid)
 		)
+		(locked yes)
 		(layer "Edge.Cuts")
 	)
@@
 	)
 	(group ""
+		(locked yes)
 		(members "08e62b6e-ce53-40d2-b3f8-55d689e35f33" "66c1f79e-09a2-49f6-90df-8659d6d0da7c"
 			"b0ed438f-358f-44be-bb09-ac3e2ab8c9ff" "b51dc32d-5a38-49bd-95bd-c49b440edd10"
 		)
 	)
+	(group ""
+		(locked yes)
+		(members "0f8eb93d-cfeb-45ff-9cf8-5a32cdc08e62" "2ae4978c-e308-4bb3-a72f-a139c856e831"
+			"378273be-b4c3-4283-b780-3fb2f34b70fd" "53012f2c-4ddc-4aed-a6c0-63cf345439d0"
+			"5341172b-f622-44a3-b415-f56a6ee28c7e" "5c7f54a5-d3c9-43e7-a6ea-d39e5f8983d7"
+			"5ffdd343-0d23-44fe-bf98-af014d9076bf" "a6add2ef-26a7-4316-bda6-bb9cbb708c9e"
+			"ba5f63c6-9f95-4c59-9e5f-23e41b57f718" "c1c05f16-14ad-44ac-84fd-890d186ede8f"
+			"c5dccf56-d6de-4789-abe4-245a405f6b0d"
+		)
+	)
