File: LF-main/LF-main/Line_kicad/line_f/line_f.kicad_pcb (KiCad board)
At the start: 2 copper layers, 135 x 150 mm, 15 parts, among them M2 Motor_DC, M3 Motor_DC, SW1 SW_SPST, SW2 SW_SPDT, SW3 SW_Push, SW4 SW_Push, U1 TB6612FNG_LINE, m1 BLACKPILL

Commit message: 7battery-center#
Parts:
- moved U1 1.38 mm to (87.8, 113.1), turned to 90 degrees

Commit message: 7battery-center#
Parts:
- moved BT1 2.09 mm to (42.0, 141.8)
- moved SW1 0.50 mm to (51.0, 161.5)
Changed lines of the file:
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@@
 	(footprint "LINE_F_FOOT_LIB:BATTERY_LINE_XT60"
 		(layer "F.Cu")
-		(at 44.0375 141.9 -90)
+		(at 41.95 141.8 -90)
 		(property "Reference" "BT1"
 			(at 0 -0.5 270)
@@
 	(footprint "LINE_F_FOOT_LIB:battery_sw"
 		(layer "F.Cu")
-		(at 51 161 -90)
+		(at 51 161.5 -90)
 		(property "Reference" "SW1"
 			(at 0.06 5.17 90)

Commit message: 7battery-center#
Parts:
- moved BT1 0.50 mm to (41.5, 141.8)
Changed lines of the file:
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@@
 	(footprint "LINE_F_FOOT_LIB:BATTERY_LINE_XT60"
 		(layer "F.Cu")
-		(at 41.95 141.8 -90)
+		(at 41.45 141.8 -90)
 		(property "Reference" "BT1"
 			(at 0 -0.5 270)
@@
 			(at 8.128 -17.018 90)
 			(layer "F.SilkS")
+			(hide yes)
 			(effects
 				(font
@@
 			(at -0.04 -23.9 0)
 			(layer "F.SilkS")
-			(effects
-				(font
+			(hide yes)
+			(effects
+				(font

Commit message: 7battery-center#
Parts:
- moved BUCK1 0.50 mm to (112.8, 138.4)
Routing:
- added copper zone on B.Cu, net C_GND
- added copper zone on F.Cu, net C_GND
Other:
- outline, holes or cut-outs redrawn
Changed lines of the file:
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@@
 	(footprint "LINE_F_FOOT_LIB:BUCK_SMD"
 		(layer "F.Cu")
-		(at 113.3375 138.437 180)
+		(at 112.8375 138.437 180)
 		(property "Reference" "BUCK1"
 			(at -11.1625 -3.563 180)
@@
 		)
 		(fp_text user "A11"
-			(at -13.3609 -7.03384 0)
+			(at -14.12 -7.09 0)
 			(unlocked yes)
 			(layer "F.SilkS")
@@
 		)
 		(fp_text user "A9"
-			(at -12.7142 -12.11384 0)
+			(at -13.4733 -12.17 0)
 			(unlocked yes)
 			(layer "F.SilkS")
@@
 		)
 		(fp_text user "A15"
-			(at -13.3609 -1.95384 0)
+			(at -14.12 -2.01 0)
 			(unlocked yes)
 			(layer "F.SilkS")
@@
 		)
 		(fp_text user "3V3"
-			(at -13.9959 23.44616 0)
+			(at -14.12 23.39 0)
 			(unlocked yes)
 			(layer "F.SilkS")
@@
 		)
 		(fp_text user "A1"
-			(at 10.7808 8.20616 0)
+			(at 11.38 8.65 0)
 			(unlocked yes)
 			(layer "F.SilkS")
@@
 		)
 		(fp_text user "B14"
-			(at -13.3609 -19.73384 0)
+			(at -14.12 -19.79 0)
 			(unlocked yes)
 			(layer "F.SilkS")
@@
 		)
 		(fp_text user "C13"
-			(at 10.7691 20.90616 0)
+			(at 11.3683 21.35 0)
 			(unlocked yes)
 			(layer "F.SilkS")
@@
 		)
 		(fp_text user "A5"
-			(at 10.7808 -1.95384 0)
+			(at 11.38 -1.51 0)
 			(unlocked yes)
 			(layer "F.SilkS")
@@
 		)
 		(fp_text user "B4"
-			(at -12.7142 3.12616 0)
+			(at -13.4733 3.07 0)
 			(unlocked yes)
 			(layer "F.SilkS")
@@
 		)
 		(fp_text user "R"
-			(at 10.795 13.29248 0)
+			(at 11.3942 13.73632 0)
 			(unlocked yes)
 			(layer "F.SilkS")
@@
 		)
 		(fp_text user "A3"
-			(at 10.7808 3.12616 0)
+			(at 11.38 3.57 0)
 			(unlocked yes)
 			(layer "F.SilkS")
@@
 		)
 		(fp_text user "B9"
-			(at -12.7142 15.82616 0)
+			(at -13.4733 15.77 0)
 			(unlocked yes)
 			(layer "F.SilkS")
@@
 		)
 		(fp_text user "B5"
-			(at -12.7142 5.66616 0)
+			(at -13.4733 5.61 0)
 			(unlocked yes)
 			(layer "F.SilkS")
@@
 		)
 		(fp_text user "B13"
-			(at -13.3609 -22.27384 0)
+			(at -14.12 -22.33 0)
 			(unlocked yes)
 			(layer "F.SilkS")
@@
 		)
 		(fp_text user "Vb"
-			(at 10.7808 23.44616 0)
+			(at 11.38 23.89 0)
 			(unlocked yes)
 			(layer "F.SilkS")
@@
 		)
 		(fp_text user "B3"
-			(at -12.7142 0.58616 0)
+			(at -13.4733 0.53 0)
 			(unlocked yes)
 			(layer "F.SilkS")
@@
 		)
 		(fp_text user "C15"
-			(at 10.7691 15.82616 0)
+			(at 11.3683 16.27 0)
 			(unlocked yes)
 			(layer "F.SilkS")
@@
 		)
 		(fp_text user "A4"
-			(at 10.7808 0.58616 0)
+			(at 11.38 1.03 0)
 			(unlocked yes)
 			(layer "F.SilkS")
@@
 		)
 		(fp_text user "5V"
-			(at 10.7808 -24.81384 0)
+			(at 11.38 -24.37 0)
 			(unlocked yes)
 			(layer "F.SilkS")
@@
 		)
 		(fp_text user "B8"
-			(at -12.7142 13.28616 0)
+			(at -13.4733 13.23 0)
 			(unlocked yes)
 			(layer "F.SilkS")
@@
 		)
 		(fp_text user "A7"
-			(at 10.7808 -7.03384 0)
+			(at 11.38 -6.59 0)
 			(unlocked yes)
 			(layer "F.SilkS")
@@
 		)
 		(fp_text user "A6"
-			(at 10.7808 -4.49384 0)
+			(at 11.38 -4.05 0)
 			(unlocked yes)
 			(layer "F.SilkS")
@@
 		)
 		(fp_text user "B6"
-			(at -12.7142 8.20616 0)
+			(at -13.4733 8.15 0)
 			(unlocked yes)
 			(layer "F.SilkS")
@@
 		)
 		(fp_text user "A12"
-			(at -13.3609 -4.49384 0)
+			(at -14.12 -4.55 0)
 			(unlocked yes)
 			(layer "F.SilkS")
@@
 		)
 		(fp_text user "G"
-			(at -12.065 20.91248 0)
+			(at -12.8241 20.85632 0)
 			(unlocked yes)
 			(layer "F.SilkS")
@@
 		)
 		(fp_text user "B12"
-			(at -13.3609 -24.81384 0)
+			(at -14.12 -24.87 0)
 			(unlocked yes)
 			(layer "F.SilkS")
@@
 		)
 		(fp_text user "A10"
-			(at -13.3609 -9.57384 0)
+			(at -14.12 -9.63 0)
 			(unlocked yes)
 			(layer "F.SilkS")
@@
 		)
 		(fp_text user "A0"
-			(at 10.7808 10.74616 0)
+			(at 11.38 11.19 0)
 			(unlocked yes)
 			(layer "F.SilkS")
@@
 		)
 		(fp_text user "B10"
-			(at 10.7691 -17.19384 0)
+			(at 11.3683 -16.75 0)
 			(unlocked yes)
 			(layer "F.SilkS")
@@
 		)
 		(fp_text user "G"
-			(at 10.795 -22.26752 0)
+			(at 11.3942 -21.82368 0)
 			(unlocked yes)
 			(layer "F.SilkS")
@@
 		)
 		(fp_text user "A8"
-			(at -12.7142 -14.65384 0)
+			(at -13.4733 -14.71 0)
 			(unlocked yes)
 			(layer "F.SilkS")
@@
 		)
 		(fp_text user "B2"
-			(at 10.7808 -14.65384 0)
+			(at 11.38 -14.21 0)
 			(unlocked yes)
 			(layer "F.SilkS")
@@
 		)
 		(fp_text user "C14"
-			(at 10.7691 18.36616 0)
+			(at 11.3683 18.81 0)
 			(unlocked yes)
 			(layer "F.SilkS")
@@
 		)
 		(fp_text user "B1"
-			(at 10.7808 -12.11384 0)
+			(at 11.38 -11.67 0)
 			(unlocked yes)
 			(layer "F.SilkS")
@@
 		)
 		(fp_text user "B7"
-			(at -12.7142 10.74616 0)
+			(at -13.4733 10.69 0)
 			(unlocked yes)
 			(layer "F.SilkS")
@@
 		)
 		(fp_text user "B15"
-			(at -13.3609 -17.19384 0)
+			(at -14.12 -17.25 0)
 			(unlocked yes)
 			(layer "F.SilkS")
@@
 		)
 		(fp_text user "5V"
-			(at -12.7142 18.36616 0)
+			(at -13.4733 18.31 0)
 			(unlocked yes)
 			(layer "F.SilkS")
@@
 		)
 		(fp_text user "B0"
-			(at 10.7808 -9.57384 0)
+			(at 11.38 -9.13 0)
 			(unlocked yes)
 			(layer "F.SilkS")
@@
 		)
 		(fp_text user "A2"
-			(at 10.7808 5.66616 0)
+			(at 11.38 6.11 0)
 			(unlocked yes)
 			(layer "F.SilkS")
@@
 		)
 		(fp_text user "3V3"
-			(at 10.7691 -19.73384 0)
+			(at 11.3683 -19.29 0)
 			(unlocked yes)
 			(layer "F.SilkS")
@@
 	)
 	(gr_circle
-		(center 87.5 59.5)
-		(end 89.024 58.738)
+		(center 87.5 58.74)
+		(end 89.203884 58.74)
 		(stroke
 			(width 0.05)
-			(type default)
+			(type solid)
 		)
 		(fill no)
@@
 		(layer "Edge.Cuts")
 	)
+	(zone
+		(net 1)
+		(net_name "C_GND")
+		(layers "F.Cu" "B.Cu")
+		(hatch edge 0.5)
+		(connect_pads
+			(clearance 0.5)
+		)
+		(min_thickness 0.25)
+		(filled_areas_thickness no)
+		(fill yes
+			(thermal_gap 0.5)
+			(thermal_bridge_width 0.5)
+		)
+		(polygon
+			(pts
+				(xy 18.5 21.5) (xy 19 174) (xy 159 173) (xy 158 21) (xy 158 20.5)
+			)
+		)
+	)
 	(group ""

Commit message: 7r-start#
Routing:
- net STBY: track 0.00 -> 59.3 mm
- net PWMB: track 0.00 -> 37.1 mm, vias 0 -> 1
- net BI2: track 0.00 -> 35.6 mm
- net BI1: track 0.00 -> 34.7 mm
- net AI1: track 0.00 -> 20.1 mm
- net AI2: track 0.00 -> 17.3 mm
- net PWMA: track 0.00 -> 0.79 mm
- removed copper zone on B.Cu, net C_GND
- removed copper zone on F.Cu, net C_GND
Other:
- outline, holes or cut-outs redrawn
Changed lines of the file:
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@@
 	)
 	(gr_arc
-		(start 67.5 107)
-		(mid 66.035534 110.535534)
-		(end 62.5 112)
+		(start 67.500001 81.999998)
+		(mid 57.707438 102.207437)
+		(end 37.5 112)
 		(stroke
 			(width 0.05)
@@
 	(gr_line
 		(start 25 112)
-		(end 62.5 112)
+		(end 37.5 112)
 		(stroke
 			(width 0.05)
@@
 	)
 	(gr_line
-		(start 67.5 107)
+		(start 67.500001 81.999995)
 		(end 67.5 47)
 		(stroke
@@
 		(layer "Edge.Cuts")
 	)
-	(zone
-		(net 1)
-		(net_name "C_GND")
+	(segment
+		(start 91.62 75.72)
+		(end 95.74 71.6)
+		(width 0.3)
+		(layer "B.Cu")
+		(net 25)
+	)
+	(segment
+		(start 91.62 105.5)
+		(end 91.62 75.72)
+		(width 0.3)
+		(layer "B.Cu")
+		(net 25)
+	)
+	(segment
+		(start 89.08 105.5)
+		(end 89.08 105.92)
+		(width 0.3)
+		(layer "F.Cu")
+		(net 29)
+	)
+	(segment
+		(start 93 101.58)
+		(end 93 76.88)
+		(width 0.3)
+		(layer "F.Cu")
+		(net 29)
+	)
+	(segment
+		(start 93 76.88)
+		(end 95.74 74.14)
+		(width 0.3)
+		(layer "F.Cu")
+		(net 29)
+	)
+	(segment
+		(start 89.08 105.5)
+		(end 93 101.58)
+		(width 0.3)
+		(layer "F.Cu")
+		(net 29)
+	)
+	(segment
+		(start 89.08 105.92)
+		(end 89 106)
+		(width 0.3)
+		(layer "F.Cu")
+		(net 29)
+	)
+	(segment
+		(start 79 105.5)
+		(end 79.5 106)
+		(width 0.3)
+		(layer "F.Cu")
+		(net 30)
+	)
+	(segment
+		(start 78.92 105.5)
+		(end 79 105.5)
+		(width 0.3)
+		(layer "F.Cu")
+		(net 30)
+	)
+	(segment
+		(start 86.54 105.5)
+		(end 86.54 79.04)
+		(width 0.3)
+		(layer "F.Cu")
+		(net 31)
+	)
+	(segment
+		(start 84.5 77)
+		(end 84.5 52.74)
+		(width 0.3)
+		(layer "F.Cu")
+		(net 31)
+	)
+	(segment
+		(start 86.54 79.04)
+		(end 84.5 77)
+		(width 0.3)
+		(layer "F.Cu")
+		(net 31)
+	)
+	(segment
+		(start 84.5 52.74)
+		(end 80.5 48.74)
+		(width 0.3)
+		(layer "F.Cu")
+		(net 31)
+	)
+	(segment
+		(start 94.16 74.66)
+		(end 94.16 70.64)
+		(width 0.3)
+		(layer "F.Cu")
+		(net 32)
+	)
+	(segment
+		(start 94.16 70.64)
+		(end 95.74 69.06)
+		(width 0.3)
+		(layer "F.Cu")
+		(net 32)
+	)
+	(via
+		(at 94.16 74.66)
+		(size 0.6)
+		(drill 0.3)
 		(layers "F.Cu" "B.Cu")
-		(hatch edge 0.5)
-		(connect_pads
-			(clearance 0.5)
-		)
-		(min_thickness 0.25)
-		(filled_areas_thickness no)
-		(fill yes
-			(thermal_gap 0.5)
-			(thermal_bridge_width 0.5)
-		)
-		(polygon
-			(pts
-				(xy 18.5 21.5) (xy 19 174) (xy 159 173) (xy 158 21) (xy 158 20.5)
-			)
-		)
+		(net 32)
+	)
+	(segment
+		(start 94.16 105.5)
+		(end 94.16 74.66)
+		(width 0.3)
+		(layer "B.Cu")
+		(net 32)
+	)
+	(segment
+		(start 84 105.5)
+		(end 84 90.34)
+		(width 0.3)
+		(layer "B.Cu")
+		(net 36)
+	)
+	(segment
+		(start 84 90.34)
+		(end 80.5 86.84)
+		(width 0.3)
+		(layer "B.Cu")
+		(net 36)
+	)
+	(segment
+		(start 81.46 105.5)
+		(end 82.45 104.51)
+		(width 0.3)
+		(layer "B.Cu")
+		(net 37)
+	)
+	(segment
+		(start 82.45 104.51)
+		(end 82.45 91.33)
+		(width 0.3)
+		(layer "B.Cu")
+		(net 37)
+	)
+	(segment
+		(start 82.45 91.33)
+		(end 80.5 89.38)
+		(width 0.3)
+		(layer "B.Cu")
+		(net 37)
 	)
 	(group ""

Commit message: 7r-start#
Connections:
- D1 pad 1: (no net) -> C_GND
- D1 pad 2: (no net) -> Net-(D1-A)
- M2 pad 1: (no net) -> AO1
- M2 pad 2: (no net) -> AO2
- M3 pad 1: (no net) -> BO1
- M3 pad 2: (no net) -> BO2
- R1 pad 1: (no net) -> LED_F
- R1 pad 2: (no net) -> Net-(D1-A)
- SW1 pad 1: (no net) -> V_SW
- SW1 pad 2: (no net) -> V_BAT
- SW2 pad 1: (no net) -> C_GND
- SW2 pad 2: (no net) -> PRIORITY_SW
- SW2 pad 3: (no net) -> S_3V3
- SW3 pad 1: (no net) -> SW_RUN
- SW3 pad 2: (no net) -> C_GND
- SW4 pad 1: (no net) -> SW_TRY
- SW4 pad 2: (no net) -> C_GND
Routing:
- net PWMA: track 0.79 -> 19.0 mm, vias 0 -> 1
Changed lines of the file:
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@@
 	(net 55 "unconnected-(U1-GND-Pad3)")
 	(net 56 "unconnected-(m1-A10-Pad7)")
+	(net 57 "Net-(D1-A)")
 	(footprint "LINE_F_FOOT_LIB:BATTERY_LINE_XT60"
 		(layer "F.Cu")
@@
 			)
 		)
+		(property ki_fp_filters "LED* LED_SMD:* LED_THT:*")
+		(sheetname "/")
+		(sheetfile "line_f.kicad_sch")
 		(attr through_hole)
 		(fp_line
@@
 			(layers "*.Cu" "*.Mask")
 			(remove_unused_layers no)
+			(net 1 "C_GND")
 			(pinfunction "K")
 			(pintype "passive")
@@
 			(layers "*.Cu" "*.Mask")
 			(remove_unused_layers no)
+			(net 57 "Net-(D1-A)")
 			(pinfunction "A")
 			(pintype "passive")
@@
 			)
 		)
+		(sheetname "/")
+		(sheetfile "line_f.kicad_sch")
 		(fp_rect
 			(start -9.36 -4.18)
@@
 			(layers "*.Cu" "*.Mask")
 			(remove_unused_layers no)
+			(net 2 "V_SW")
 			(pinfunction "A")
 			(pintype "passive")
@@
 			(layers "*.Cu" "*.Mask")
 			(remove_unused_layers no)
+			(net 3 "V_BAT")
 			(pinfunction "B")
 			(pintype "passive")
@@
 			)
 		)
+		(property ki_fp_filters "PinHeader*P2.54mm* TerminalBlock*")
+		(sheetname "/")
+		(sheetfile "line_f.kicad_sch")
 		(attr through_hole)
 		(fp_line
@@
 			(remove_unused_layers no)
 			(roundrect_rratio 0.147059)
+			(net 46 "AO1")
 			(pinfunction "+")
 			(pintype "passive")
@@
 			(layers "*.Cu" "*.Mask")
 			(remove_unused_layers no)
+			(net 47 "AO2")
 			(pinfunction "-")
 			(pintype "passive")
@@
 			)
 		)
+		(property ki_fp_filters "PinHeader*P2.54mm* TerminalBlock*")
+		(sheetname "/")
+		(sheetfile "line_f.kicad_sch")
 		(attr through_hole)
 		(fp_line
@@
 			(remove_unused_layers no)
 			(roundrect_rratio 0.147059)
+			(net 48 "BO1")
 			(pinfunction "+")
 			(pintype "passive")
@@
 			(layers "*.Cu" "*.Mask")
 			(remove_unused_layers no)
+			(net 49 "BO2")
 			(pinfunction "-")
 			(pintype "passive")
@@
 			)
 		)
+		(property ki_fp_filters "R_*")
+		(sheetname "/")
+		(sheetfile "line_f.kicad_sch")
 		(attr through_hole)
 		(fp_line
@@
 			(layers "*.Cu" "*.Mask")
 			(remove_unused_layers no)
+			(net 41 "LED_F")
 			(pintype "passive")
 		)
@@
 			(layers "*.Cu" "*.Mask")
 			(remove_unused_layers no)
+			(net 57 "Net-(D1-A)")
 			(pintype "passive")
 		)
@@
 			)
 		)
+		(sheetname "/")
+		(sheetfile "line_f.kicad_sch")
 		(attr through_hole)
 		(fp_rect
@@
 			(layers "*.Cu" "*.Mask")
 			(remove_unused_layers no)
+			(net 43 "SW_RUN")
 			(pinfunction "1")
 			(pintype "passive")
@@
 			(layers "*.Cu" "*.Mask")
 			(remove_unused_layers no)
+			(net 43 "SW_RUN")
 			(pinfunction "1")
 			(pintype "passive")
@@
 			(layers "*.Cu" "*.Mask")
 			(remove_unused_layers no)
+			(net 1 "C_GND")
 			(pinfunction "2")
 			(pintype "passive")
@@
 			(layers "*.Cu" "*.Mask")
 			(remove_unused_layers no)
+			(net 1 "C_GND")
 			(pinfunction "2")
 			(pintype "passive")
@@
 			)
 		)
+		(sheetname "/")
+		(sheetfile "line_f.kicad_sch")
 		(attr through_hole)
 		(fp_rect
@@
 			(chamfer_ratio 0.2)
 			(chamfer top_left)
+			(net 1 "C_GND")
 			(pinfunction "A")
 			(pintype "passive")
@@
 			(layers "*.Cu" "*.Mask")
 			(remove_unused_layers no)
+			(net 22 "PRIORITY_SW")
 			(pinfunction "B")
 			(pintype "passive")
@@
 			(layers "*.Cu" "*.Mask")
 			(remove_unused_layers no)
+			(net 33 "S_3V3")
 			(pinfunction "C")
 			(pintype "passive")
@@
 			)
 		)
+		(sheetname "/")
+		(sheetfile "line_f.kicad_sch")
 		(attr through_hole)
 		(fp_rect
@@
 			(layers "*.Cu" "*.Mask")
 			(remove_unused_layers no)
+			(net 40 "SW_TRY")
 			(pinfunction "1")
 			(pintype "passive")
@@
 			(layers "*.Cu" "*.Mask")
 			(remove_unused_layers no)
+			(net 40 "SW_TRY")
 			(pinfunction "1")
 			(pintype "passive")
@@
 			(layers "*.Cu" "*.Mask")
 			(remove_unused_layers no)
+			(net 1 "C_GND")
 			(pinfunction "2")
 			(pintype "passive")
@@
 			(layers "*.Cu" "*.Mask")
 			(remove_unused_layers no)
+			(net 1 "C_GND")
 			(pinfunction "2")
 			(pintype "passive")
@@
 	)
 	(segment
+		(start 85.5 98.92)
+		(end 85.5 90)
+		(width 0.3)
+		(layer "F.Cu")
+		(net 30)
+	)
+	(segment
 		(start 78.92 105.5)
 		(end 79 105.5)
@@
 		(net 30)
 	)
+	(segment
+		(start 78.92 105.5)
+		(end 85.5 98.92)
+		(width 0.3)
+		(layer "F.Cu")
+		(net 30)
+	)
+	(via
+		(at 85.5 90)
+		(size 0.6)
+		(drill 0.3)
+		(layers "F.Cu" "B.Cu")
+		(net 30)
+	)
