File: LF-main/LF-main/Line_kicad/line_f/line_f.kicad_pcb (KiCad board)
At the start: 2 copper layers, 135 x 150 mm, 15 parts, among them M2 Motor_DC, M3 Motor_DC, SW1 SW_SPST, SW2 SW_SPDT, SW3 SW_Push, SW4 SW_Push, U1 TB6612FNG_LINE, m1 BLACKPILL

Commit message: 7r-start#
Parts:
- moved M3 92.0 mm to (128.9, 163.6)
- moved M2 91.6 mm to (46.5, 163.4)
- moved SW1 73.0 mm to (124.0, 161.5)
- moved SW2 28.0 mm to (90.9, 171.3)
- moved BUCK1 6.00 mm to (112.8, 132.4)
Changed lines of the file:
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@@
 	(footprint "LINE_F_FOOT_LIB:BUCK_SMD"
 		(layer "F.Cu")
-		(at 112.8375 138.437 180)
+		(at 112.8375 132.437 180)
 		(property "Reference" "BUCK1"
 			(at -11.1625 -3.563 180)
@@
 	(footprint "LINE_F_FOOT_LIB:battery_sw"
 		(layer "F.Cu")
-		(at 51 161.5 -90)
+		(at 124 161.5 -90)
 		(property "Reference" "SW1"
 			(at 0.06 5.17 90)
@@
 	(footprint "LINE_F_FOOT_LIB:connector_motor"
 		(layer "F.Cu")
-		(at 138.09 163.39 90)
+		(at 46.48 163.39 90)
 		(property "Reference" "M2"
 			(at 0 -0.5 90)
@@
 	(footprint "LINE_F_FOOT_LIB:connector_motor"
 		(layer "F.Cu")
-		(at 36.91 163.61 -90)
+		(at 128.91 163.61 -90)
 		(property "Reference" "M3"
 			(at 0 -0.5 270)
@@
 	(footprint "LINE_F_FOOT_LIB:SLIDE SW"
 		(layer "F.Cu")
-		(at 62.91 171.3125)
+		(at 90.91 171.3125)
 		(property "Reference" "SW2"
 			(at -6.94 -3.79 0)

Commit message: 7r-start#
Parts:
- moved SW2 3.46 mm to (87.5, 171.3)
Changed lines of the file:
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@@
 	(footprint "LINE_F_FOOT_LIB:SLIDE SW"
 		(layer "F.Cu")
-		(at 90.91 171.3125)
+		(at 87.45 171.3125)
 		(property "Reference" "SW2"
 			(at -6.94 -3.79 0)

Commit message: 7r-start.5#
Parts:
- moved BUCK1 28.1 mm to (140.0, 139.6), turned to 0 degrees
- moved D1 10.3 mm to (148.8, 111.6), turned to 180 degrees
Routing:
- net SW_RUN: track 0.00 -> 162.2 mm, vias 0 -> 2
- net V_BAT: track 0.00 -> 155.6 mm
- net SW_TRY: track 0.00 -> 153.7 mm, vias 0 -> 1
- net S_3V3: track 0.00 -> 138.9 mm, vias 0 -> 1
- net LSA_TX: track 0.00 -> 111.3 mm, vias 0 -> 2
- net D7: track 0.00 -> 109.4 mm, vias 0 -> 1
- net LSA_RX: track 0.00 -> 106.8 mm, vias 0 -> 2
- net 5V: track 0.00 -> 104.9 mm
- net PRIORITY_SW: track 0.00 -> 104.6 mm, vias 0 -> 1
- net D6: track 0.00 -> 101.6 mm, vias 0 -> 2
- net LED_F: track 0.00 -> 92.3 mm, vias 0 -> 1
- net D5: track 0.00 -> 86.2 mm, vias 0 -> 1
- net LSA_UEN: track 0.00 -> 85.3 mm, vias 0 -> 1
- net AO2: track 0.00 -> 83.8 mm, vias 0 -> 1
- net AO1: track 0.00 -> 83.5 mm, vias 0 -> 1
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
Commit message: 7r-start.5#
Routing:
- added copper zone on B.Cu, net C_GND
- added copper zone on F.Cu, net C_GND
Changed lines of the file:
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@@
 		(net 57)
+	)
+	(zone
+		(net 1)
+		(net_name "C_GND")
+		(layers "F.Cu" "B.Cu")
+		(hatch edge 0.5)
+		(connect_pads
+			(clearance 0.5)
+		)
+		(min_thickness 0.25)
+		(filled_areas_thickness no)
+		(fill
+			(thermal_gap 0.5)
+			(thermal_bridge_width 0.5)
+		)
+		(polygon
+			(pts
+				(xy 156.5 172) (xy 156.5 21.5) (xy 18.5 21.5) (xy 17 23) (xy 17 172) (xy 18 173) (xy 155.5 173)
+			)
+		)
 	)
 	(embedded_fonts no)
