File: LF-main/LF-main/Line_kicad/line_f/line_f.kicad_pcb (KiCad board)
At the start: 2 copper layers, 135 x 150 mm, 16 parts, among them M2 Motor_DC, M3 Motor_DC, M4 NOT_MOTOR, SW1 SW_SPST, SW2 SW_SPDT, SW3 SW_Push, SW4 SW_Push, U1 TB6612FNG_LINE, m1 BLACKPILL

Commit message: 7r-start.77#
Routing:
- net BO2: track 80.6 -> 64.6 mm, vias 1 -> 0
- net AO2: track 83.8 -> 83.1 mm
Changed lines of the file:
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@@
 	)
 	(segment
-		(start 42 162.21)
-		(end 42 160.908)
+		(start 45.363 158.847)
+		(end 42 162.21)
 		(width 0.5)
 		(layer "B.Cu")
@@
 	)
 	(segment
-		(start 42 160.908)
-		(end 44.0613 158.847)
-		(width 0.5)
-		(layer "B.Cu")
-		(net 47)
-	)
-	(segment
-		(start 44.0613 158.847)
-		(end 83.0944 158.847)
+		(start 83.0944 158.847)
+		(end 45.363 158.847)
 		(width 0.5)
 		(layer "B.Cu")
@@
 	)
 	(segment
-		(start 93.27 122.39)
-		(end 93.27 157.486)
-		(width 0.5)
-		(layer "F.Cu")
-		(net 49)
-	)
-	(segment
-		(start 91.62 120.74)
-		(end 93.27 122.39)
-		(width 0.5)
-		(layer "F.Cu")
-		(net 49)
-	)
-	(via
-		(at 93.27 157.486)
-		(size 0.6)
-		(drill 0.3)
-		(layers "F.Cu" "B.Cu")
-		(net 49)
-	)
-	(segment
-		(start 93.27 157.486)
-		(end 126.086 157.486)
+		(start 125.97868 157.37868)
+		(end 133.39 164.79)
 		(width 0.5)
 		(layer "B.Cu")
@@
 	)
 	(segment
-		(start 126.086 157.486)
-		(end 133.39 164.79)
+		(start 111 141.362641)
+		(end 111 146.5)
 		(width 0.5)
 		(layer "B.Cu")
+		(net 49)
+	)
+	(segment
+		(start 91.62 120.74)
+		(end 110.121321 139.241321)
+		(width 0.5)
+		(layer "B.Cu")
+		(net 49)
+	)
+	(segment
+		(start 121 156.5)
+		(end 123.857359 156.5)
+		(width 0.5)
+		(layer "B.Cu")
+		(net 49)
+	)
+	(arc
+		(start 125.97868 157.37868)
+		(mid 125.00541 156.728361)
+		(end 123.857359 156.5)
+		(width 0.5)
+		(layer "B.Cu")
+		(net 49)
+	)
+	(arc
+		(start 121 156.5)
+		(mid 113.928932 153.571068)
+		(end 111 146.5)
+		(width 0.5)
+		(layer "B.Cu")
+		(net 49)
+	)
+	(arc
+		(start 110.121321 139.241321)
+		(mid 110.771639 140.214591)
+		(end 111 141.362641)
+		(width 0.5)
+		(layer "B.Cu")

Commit message: 7r-start.77#
Routing:
- net AO1: track 83.5 -> 63.0 mm
- net AO2: track 83.1 -> 64.3 mm, vias 1 -> 2
Changed lines of the file:
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@@
 	)
 	(segment
-		(start 43.5105 163.24)
-		(end 43.5105 127.824)
+		(start 67.39 139.89)
+		(end 42.53 164.75)
 		(width 0.5)
 		(layer "F.Cu")
@@
 	)
 	(segment
-		(start 42 164.75)
-		(end 43.5105 163.24)
+		(start 42.53 164.75)
+		(end 42 164.75)
 		(width 0.5)
 		(layer "F.Cu")
@@
 	)
 	(via
-		(at 43.5105 127.824)
+		(at 67.39 139.89)
 		(size 0.6)
 		(drill 0.3)
@@
 	)
 	(segment
-		(start 86.54 120.74)
-		(end 79.4564 127.824)
+		(start 67.39 139.89)
+		(end 67.231 140.049)
 		(width 0.5)
 		(layer "B.Cu")
@@
 	)
 	(segment
-		(start 79.4564 127.824)
-		(end 43.5105 127.824)
+		(start 86.54 120.74)
+		(end 67.39 139.89)
 		(width 0.5)
 		(layer "B.Cu")
@@
 	)
 	(segment
-		(start 83.0944 126.726)
-		(end 83.0944 158.847)
-		(width 0.5)
-		(layer "F.Cu")
-		(net 47)
-	)
-	(segment
-		(start 89.08 120.74)
-		(end 83.0944 126.726)
+		(start 66.66 143.16)
+		(end 54.41 155.41)
 		(width 0.5)
 		(layer "F.Cu")
@@
 	)
 	(via
-		(at 83.0944 158.847)
+		(at 54.41 155.41)
+		(size 0.6)
+		(drill 0.3)
+		(layers "F.Cu" "B.Cu")
+		(net 47)
+	)
+	(via
+		(at 66.66 143.16)
 		(size 0.6)
 		(drill 0.3)
@@
 	)
 	(segment
-		(start 45.363 158.847)
+		(start 47.61 162.21)
 		(end 42 162.21)
 		(width 0.5)
@@
 	)
 	(segment
-		(start 83.0944 158.847)
-		(end 45.363 158.847)
+		(start 89.08 120.74)
+		(end 66.66 143.16)
 		(width 0.5)
 		(layer "B.Cu")
+		(net 47)
+	)
+	(segment
+		(start 54.41 155.41)
+		(end 47.61 162.21)
+		(width 0.5)
+		(layer "B.Cu")

Commit message: 7r-start.77#
Changed lines of the file:
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@@
 	)
 	(segment
-		(start 127.5 156.36)
+		(start 128.37868 157.23868)
 		(end 133.39 162.25)
 		(width 0.5)
@@
 	(segment
 		(start 127.5 138.539)
-		(end 127.5 156.36)
+		(end 127.5 155.117359)
 		(width 0.5)
 		(layer "F.Cu")
@@
 		(net 48)
 	)
+	(arc
+		(start 127.5 155.117359)
+		(mid 127.728362 156.26541)
+		(end 128.37868 157.23868)
+		(width 0.5)
+		(layer "F.Cu")
+		(net 48)
+	)
 	(segment
-		(start 111.959 138.539)
+		(start 113.201641 138.539)
 		(end 127.5 138.539)
 		(width 0.5)
@@
 	(segment
 		(start 94.16 120.74)
-		(end 111.959 138.539)
+		(end 111.080321 137.660321)
 		(width 0.5)
 		(layer "B.Cu")
+		(net 48)
+	)
+	(arc
+		(start 113.201641 138.539)
+		(mid 112.053591 138.310639)
+		(end 111.080321 137.660321)
+		(width 0.5)
+		(layer "B.Cu")

Commit message: 7r-start.77#
Changed lines of the file:
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@@
 	(segment
 		(start 122.736 127.011)
-		(end 111.63 115.906)
+		(end 112.655107 116.931015)
 		(width 0.5)
 		(layer "B.Cu")
@@
 	)
 	(segment
-		(start 111.63 115.906)
-		(end 83.7545 115.906)
+		(start 110.180345 115.906)
+		(end 85.204141 115.906)
 		(width 0.5)
 		(layer "B.Cu")
@@
 	)
 	(segment
-		(start 83.7545 115.906)
+		(start 82.729395 116.930999)
 		(end 78.92 120.74)
 		(width 0.5)
@@
 		(net 3)
 	)
+	(arc
+		(start 82.729395 116.930999)
+		(mid 83.864832 116.172387)
+		(end 85.204141 115.906)
+		(width 0.5)
+		(layer "B.Cu")
+		(net 3)
+	)
+	(arc
+		(start 112.655107 116.931015)
+		(mid 111.519664 116.172392)
+		(end 110.180345 115.906)
+		(width 0.5)
+		(layer "B.Cu")
+		(net 3)
+	)
 	(segment
 		(start 95.74 48.74)
@@
 	)
 	(segment
-		(start 85.4773 116.723)
+		(start 86.926971 116.723)
 		(end 100.774 116.723)
 		(width 0.5)
@@
 	(segment
 		(start 81.46 120.74)
-		(end 85.4773 116.723)
-		(width 0.5)
-		(layer "B.Cu")
+		(end 84.45219 117.748034)
+		(width 0.5)
+		(layer "B.Cu")
+		(net 33)
+	)
+	(arc
+		(start 84.45219 117.748034)
+		(mid 85.58764 116.989397)
+		(end 86.926971 116.723)
+		(width 0.5)
+		(layer "B.Cu")
