File: LF-main/LF-main/Line_kicad/line_f/line_f.kicad_sch (KiCad schematic)
At the start: 15 parts, among them M2 Motor_DC, M3 Motor_DC, SW1 SW_SPST, SW2 SW_SPDT, SW3 SW_Push, SW4 SW_Push, U1 TB6612FNG_LINE, m1 BLACKPILL

Commit message: 7r-start.5#
Parts:
- added M4: NOT_MOTOR, LINE_F_FOOT_LIB:connector_motor, symbol Motor:Motor_DC
Connections:
- net 5V: now also M4.1 (+)
- net C_GND: now also M4.2 (-)
Changed lines of the file:
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@@
+		)
+	)
+	(global_label "C_GND"
+		(shape input)
+		(at 127 67.31 0)
+		(fields_autoplaced yes)
+		(effects
+			(font
+				(size 1.27 1.27)
+			)
+			(justify left)
+		)
+		(property "Intersheetrefs" "${INTERSHEET_REFS}"
+			(at 136.0933 67.31 0)
+			(effects
+				(font
+					(size 1.27 1.27)
+				)
+				(justify left)
+				(hide yes)
+			)
 		)
 	)
@@
 		(property "Intersheetrefs" "${INTERSHEET_REFS}"
 			(at 167.64 82.7533 90)
+			(effects
+				(font
+					(size 1.27 1.27)
+				)
+				(justify right)
+				(hide yes)
+			)
+		)
+	)
+	(global_label "5V"
+		(shape input)
+		(at 114.3 67.31 180)
+		(fields_autoplaced yes)
+		(effects
+			(font
+				(size 1.27 1.27)
+			)
+			(justify right)
+		)
+		(property "Intersheetrefs" "${INTERSHEET_REFS}"
+			(at 109.0167 67.31 0)
 			(effects
 				(font
@@
 					(unit 1)
 				)
+			)
+		)
+	)
+	(symbol
+		(lib_id "Motor:Motor_DC")
+		(at 119.38 67.31 90)
+		(unit 1)
+		(exclude_from_sim no)
+		(in_bom yes)
+		(on_board yes)
+		(dnp no)
+		(property "Reference" "M4"
+			(at 126.238 63.5 90)
+			(effects
+				(font
+					(size 1.27 1.27)
+				)
+				(justify left)
+			)
+		)
+		(property "Value" "NOT_MOTOR"
+			(at 126.238 60.96 90)
+			(effects
+				(font
+					(size 1.27 1.27)
+				)
+				(justify left)
+			)
+		)
+		(property "Footprint" "LINE_F_FOOT_LIB:connector_motor"
+			(at 121.666 67.31 0)
+			(effects
+				(font
+					(size 1.27 1.27)
+				)
+				(hide yes)
+			)
+		)
+		(property "Datasheet" "~"
+			(at 121.666 67.31 0)
+			(effects
+				(font
+					(size 1.27 1.27)
+				)
+				(hide yes)
+			)
+		)
+		(property "Description" "DC Motor"
+			(at 119.38 67.31 0)
+			(effects
+				(font
+					(size 1.27 1.27)
+				)
+				(hide yes)
+			)
+		)
+		(pin "1"
+		)
+		(pin "2"
+		)
+		(instances
+			(project "line_f"
+				(path "/c13c4e87-a023-4a7d-8b82-fe1a380f0003"
+					(reference "M4")
+					(unit 1)
+				)
